Commit message: Add: namespaces por robot para simular dos agentes aislados
Prepara el sistema para el esquema colaborativo de dos robots (OE2): con
'namespace' vacio el comportamiento es identico al original de un solo robot,
y con 'robot1'/'robot2' todo el grafo cuelga del namespace correspondiente.

Puntos no evidentes:

- Los plugins de Gazebo llevan sufijo de namespace en el atributo 'name'
  ('sufijo_ns' en deepracer.xacro). gazebo_ros guarda un registro estatico y
  global de nombres de nodo SIN el namespace, asi que dos robots con el mismo
  nombre de plugin comparten nodo y el segundo acaba suscrito a los topicos
  del primero.

- agent_control.yaml usa el comodin '/**', que casa con cero o mas niveles de
  namespace. Un solo archivo sirve para uno o para dos agentes.

- Los plugins que no heredan namespace de spawn_entity.py (gazebo_ros2_control,
  drive, lidar y camara) lo declaran en su propio bloque <ros>, emitido solo
  cuando el argumento trae valor para no alterar el URDF de un robot.

File: Robot/aws-deepracer/deepracer_description/models/xacro/control/deepracer_ros_control.xacro (robot description, xacro)
@@ -14,5 +14,16 @@
 <robot name="agent" xmlns:xacro="http://www.ros.org/wiki/xacro">
   <gazebo>
-      <plugin name='gazebo_ros_deepracer_drive' filename='libgazebo_ros_deepracer_drive.so'>
+      <!-- El sufijo hace unico el nombre del nodo entre robots; ver 'sufijo_ns'
+           en deepracer.xacro. Sin el, el plugin del segundo robot reutiliza el
+           nodo del primero y se suscribe a /robot1/cmd_vel. -->
+      <plugin name='gazebo_ros_deepracer_drive${sufijo_ns}' filename='libgazebo_ros_deepracer_drive.so'>
+        <!-- El plugin llama a gazebo_ros::Node::Get(_sdf), que lee este bloque.
+             Sin el, /cmd_vel y /odom se quedan en la raiz aunque el resto del
+             robot este bajo namespace. Vacio por defecto: no se emite. -->
+        <xacro:if value="${'$(arg robot_namespace)' != ''}">
+          <ros>
+            <namespace>$(arg robot_namespace)</namespace>
+          </ros>
+        </xacro:if>
         <update_rate>15.0</update_rate>
         <!-- Max absolute steer angle for tyre in radians-->
@@ -29,6 +40,7 @@
         <publish_odom>true</publish_odom>
         <publish_odom_tf>true</publish_odom_tf>
-        <odometry_frame>odom</odometry_frame>
-        <robot_base_frame>base_link</robot_base_frame>
+        <!-- Este plugin ignora el frame_prefix de robot_state_publisher. -->
+        <odometry_frame>$(arg frame_prefix)odom</odometry_frame>
+        <robot_base_frame>$(arg frame_prefix)base_link</robot_base_frame>
       </plugin>
   </gazebo>
@@ -71,5 +83,14 @@
   </ros2_control>
   <gazebo>
-    <plugin filename="libgazebo_ros2_control.so" name="gazebo_ros2_control">
+    <plugin filename="libgazebo_ros2_control.so" name="gazebo_ros2_control${sufijo_ns}">
+      <!-- Este plugin no es un plugin de gazebo_ros: no hereda el
+           -robot_namespace de spawn_entity.py. Su namespace se declara aqui.
+           El bloque solo se emite si el argumento trae valor, de modo que con
+           un robot el URDF sale byte a byte igual al original. -->
+      <xacro:if value="${'$(arg robot_namespace)' != ''}">
+        <ros>
+          <namespace>$(arg robot_namespace)</namespace>
+        </ros>
+      </xacro:if>
       <robot_param>robot_description</robot_param>
       <robot_param_node>robot_state_publisher</robot_param_node>

File: Robot/aws-deepracer/deepracer_description/models/xacro/deepracer/deepracer.xacro (robot description, xacro)
@@ -15,4 +15,18 @@
   <!-- agent argument from python xacro call-->
   <xacro:arg name="agent_name" default="agent" />
+  <!-- Prefijo de marcos TF (CONTRATO_INTERFACES.md §3). Vacio por defecto: con
+       un solo robot el URDF generado es identico al original. Con dos robots se
+       pasa 'robot1/' y 'robot2/' para que los 13 marcos dejen de colisionar.
+       Debe terminar en '/' porque se concatena tal cual.
+       Los marcos que declara el URDF (base_link, chassis, laser, ...) los
+       prefija robot_state_publisher con su parametro frame_prefix; estos tres
+       los escriben plugins de Gazebo, que lo ignoran, y hay que pasarselos. -->
+  <xacro:arg name="frame_prefix" default="" />
+  <!-- Namespace ROS 2 del agente (CONTRATO_INTERFACES.md §6). Vacio por defecto:
+       con un solo robot el URDF generado es identico al original. El plugin
+       gazebo_ros2_control no es un plugin de gazebo_ros, asi que no hereda el
+       -robot_namespace de spawn_entity.py: lee su propio bloque <ros><namespace>,
+       y por eso hay que pasarselo por aqui. Sin barra final: ROS 2 la agrega. -->
+  <xacro:arg name="robot_namespace" default="" />
   <!-- Default: Use front facing camera and LiDAR sensor -->
   <xacro:arg name="sensor_type" default="front_facing_camera_and_lidar" />
@@ -35,4 +49,15 @@
   <xacro:property name="sensor_type_val" value="$(arg sensor_type)" />
   <xacro:property name="shell_val" value="$(arg shell)" />
+  <!-- Sufijo para el atributo 'name' de los <plugin> de Gazebo.
+       gazebo_ros mantiene un registro ESTATICO Y GLOBAL de nombres de nodo
+       (gazebo_ros/node.hpp, 'static_existing_nodes_') y guarda el nombre PELADO,
+       sin namespace. El nombre sale del atributo 'name' del <plugin>. Si los dos
+       robots usan el mismo, al cargar el segundo gazebo_ros::Node::Get() ve el
+       nombre ocupado y devuelve el nodo del PRIMERO: el plugin de robot2 acaba
+       suscrito a /robot1/cmd_vel. El propio libgazebo_ros_node.so lo avisa:
+       "Found multiple nodes with same name... Try changing one of the plugin
+       names". Cambiar solo el namespace NO basta, porque el registro no lo mira.
+       Vacio sin namespace: los nombres quedan exactamente como en el original. -->
+  <xacro:property name="sufijo_ns" value="${'_$(arg robot_namespace)' if '$(arg robot_namespace)' else ''}" />
   <!-- agent macro -->
   <xacro:include filename="$(find deepracer_description)/models/xacro/macro/macros.xacro" />

File: Robot/aws-deepracer/deepracer_description/models/xacro/sensor/deepracer_gazebo_front_facing_camera.xacro (robot description, xacro)
@@ -29,5 +29,16 @@
         </clip>
       </camera>
-      <plugin name="camera_controller" filename="libgazebo_ros_camera.so">
+      <!-- El sufijo da un nombre de nodo unico entre robots (ver 'sufijo_ns' en
+           deepracer.xacro). Vacio sin namespace.
+           Cuidado con los comentarios que sobreviven al renderizado. launch_ros
+           pasa el URDF por un parser YAML, y unos dos puntos seguidos de espacio
+           lo rompen con "Unable to parse the value of parameter
+           robot_description as yaml". -->
+      <plugin name="camera_controller${sufijo_ns}" filename="libgazebo_ros_camera.so">
+        <xacro:if value="${'$(arg robot_namespace)' != ''}">
+          <ros>
+            <namespace>$(arg robot_namespace)</namespace>
+          </ros>
+        </xacro:if>
         <alwaysOn>true</alwaysOn>
         <updateRate>60</updateRate>

File: Robot/aws-deepracer/deepracer_description/models/xacro/sensor/deepracer_gazebo_lidar.xacro (robot description, xacro)
@@ -41,11 +41,17 @@
         <frameName>laser</frameName>
       </plugin>-->
-       <plugin name="rp_lidar" filename="libgazebo_ros_ray_sensor.so">
+       <!-- El sufijo da un nombre de nodo unico entre robots (ver 'sufijo_ns'
+            en deepracer.xacro). Vacio sin namespace. -->
+       <plugin name="rp_lidar${sufijo_ns}" filename="libgazebo_ros_ray_sensor.so">
           <ros>
-            <!-- <namespace>/laser</namespace> -->
+            <!-- Con namespace, '~/out' es /robot1/rp_lidar_robot1/out y el
+                 remapeo a 'scan' (relativo) lo resuelve a /robot1/scan. -->
+            <xacro:if value="${'$(arg robot_namespace)' != ''}">
+              <namespace>$(arg robot_namespace)</namespace>
+            </xacro:if>
             <argument>~/out:=scan</argument>
           </ros>
           <output_type>sensor_msgs/LaserScan</output_type>
-          <frame_name>laser</frame_name>
+          <frame_name>$(arg frame_prefix)laser</frame_name>
         </plugin>
     </sensor>
